File: mks_wifi.sch (KiCad schematic (older format))
At the start: 3 parts, among them J1 Conn_01x08, J2 Conn_01x08

Commit message: v1, проверенный вариант
Parts:
- added C1, C2: 47pF, Capacitor_SMD:C_0805_2012Metric, symbol Device:C_Small
- added C3, C5: 0.1uF, Capacitor_SMD:C_0805_2012Metric, symbol Device:C_Small
- added C4: 4.7uF, Capacitor_SMD:C_0805_2012Metric, symbol Device:C_Small
- added C6: 0.01uF, Capacitor_SMD:C_0805_2012Metric, symbol Device:C_Small
- added C7, C8: 1uF, Capacitor_SMD:C_0805_2012Metric, symbol Device:C_Small
- added J3: USB, Connector_JST:JST_XH_B4B-XH-A_1x04_P2.50mm_Vertical, symbol Connector_Generic:Conn_01x04
- added J4: UART, Connector_JST:JST_XH_B4B-XH-A_1x04_P2.50mm_Vertical, symbol Connector_Generic:Conn_01x04
- added R1, R2: 27, Resistor_SMD:R_0805_2012Metric, symbol Device:R_Small
- added U2: ISO7721, Package_SO:SOIC-8_3.9x4.9mm_P1.27mm, symbol iso7721:ISO7721
- gave numbers to parts that had none: 1
Connections:
- net GND: now also C1.2, C2.1, C3.2, C4.2, C5.2, C6.1, C7.2, J3.1 (Pin_1), J4.4 (Pin_4), U2.4 (GND1); no longer J2.8 (Pin_8)
- net RX: now also U2.7 (INA)
- net TX: now also U2.6 (OUTB)
- net 3V3: now reaches J1.8 (Pin_8)
- net 3V3: now also C8.1, U2.8 (VCC2)
- net at U1.1 (TXD): now also J4.3 (Pin_3), U2.3 (INB)
- net VDD_USB: now reaches U1.11 (~RESET)
- net VDD_USB: now also U1.12 (VCC), U1.3 (VCCIO), C3.1, C4.1, C5.1, C6.2, C7.1, J3.4 (Pin_4), J4.1 (Pin_1), U2.1 (VCC1)
- net at U1.4 (RXD): now also J4.2 (Pin_2), U2.2 (OUTA)
- net at U1.8 (USBDP): now also R2.1
- net at U1.9 (USBDM): now also R1.1
- new net GND2: C8.2, J2.8 (Pin_8), U2.5 (GND2)
- new net USB_DM: C1.1, J3.3 (Pin_3), R1.2
- new net USB_DP: C2.2, J3.2 (Pin_2), R2.2
- no-connect marks 0 -> 19
Other:
- moved on the sheet: J1, J2, U1
